File: projects/HackerPCBNameTag/src/HackerBadgePCBV2.kicad_sch (KiCad schematic)
At the start: 31 parts, among them Q1 S8050, Q2 FS8205, U1 NT3H2111W0FHKH, U2 TPS61023DRLR, U3 DW01A_C351410

Commit message: some updates
Parts:
- removed Q2: FS8205, easyeda2kicad:SOT-23-6_L2.9-W1.6-P0.95-LS2.8-BR, symbol FS8205
- added Q3: FS8205A, easyeda2kicad:SOT-23-6_L2.9-W1.6-P0.95-LS2.8-BR, symbol easyeda2kicad:FS8205A_C908265
- LED2, LED3: LCSC Part (none) -> C965815
Connections:
- net BAT-: now also Q3.3 (S2)
- net GND: now also Q3.1 (S1)
- net OC: now also Q3.6 (G1)
- net unconnected-(SWITCH1-Pad4)_1_1_1: now reaches SWITCH1.4
- net at U3.1 (OD): now also Q3.4 (G2)
