File: projects/Water Quality Checker/src/design.sch (EAGLE design)
At the start: 35 parts, among them Q2 NPN, U1 LM358_SOIC, U2 TPS61073

Commit message: update files
Signed-off-by: Shreyans Jain <shreyans@shreyans.sh>
Parts:
- added R10, R11, R4, R7, R8, R9: 150R, Resistor:R_CHIP-0402(1005-METRIC)
- added R12: 200R, Resistor:R_CHIP-0402(1005-METRIC)
- added R13, R14, R15: 200K, Resistor:R_CHIP-0402(1005-METRIC)
- L1: value 4.7µH -> 10µH
- R20: value 680R -> 470R
- R5: value 1.6M -> 1M
Connections:
- removed net N$15: R5.1, R6.2, U2.FB
- new net N$17: R4.2, U$1.1
- new net N$18: R7.2, U$1.2
- new net N$19: R8.2, U$1.4
- new net N$20: R9.2, U$1.5
- new net N$21: R10.1, TDS_R.A
- new net N$22: R11.2, U$1.7
- new net N$23: R12.1, R20.2
- new net N$24: R13.2, R5.1
- new net N$25: R13.1, R14.2
- new net N$26: R14.1, R15.2
- new net N$27: R15.1, R6.2, U2.FB
- net N$10: now also R8.1; no longer U$1.4
- net N$11: now also R9.1; no longer U$1.5
- net N$12: now also R11.1; no longer U$1.7
- net N$13: now also R10.2; no longer TDS_R.A
- net N$45: now also R12.2; no longer R20.2
- net N$8: now also R4.1; no longer U$1.1
- net N$9: now also R7.1; no longer U$1.2
Other:
- moved on the sheet: C2, R20, R23, R5, R6
