File: projects/Nat3z_65_Keyboard/src/keypad.kicad_pcb (KiCad board)
At the start: 2 copper layers, 310.8 x 106.1 mm, 150 parts, among them J1 USB_C_Receptacle, SW1 SW_Push, SW10 SW_Push, SW11 SW_Push, SW12 SW_Push, SW13 SW_Push, SW14 SW_Push, SW15 SW_Push, SW16 SW_Push, SW17 SW_Push, SW18 SW_Push, SW19 SW_Push, SW2 SW_Push, SW20 SW_Push, SW22 SW_Push, SW23 SW_Push, SW24 SW_Push, SW25 SW_Push, SW26 SW_Push, SW27 SW_Push, SW28 SW_Push, SW29 SW_Push, SW3 SW_Push, SW30 SW_Push, SW31 SW_Push, SW32 SW_Push, SW33 SW_Push, SW34 SW_Push, SW35 SW_Push, SW36 SW_Push, SW37 SW_Push, SW38 SW_Push, SW39 SW_Push, SW4 SW_Push, SW40 SW_Push, SW41 SW_Push, SW42 SW_Push, SW43 SW_Push, SW44 SW_Push, SW45 SW_Push, SW46 SW_Push, SW47 SW_Push, SW48 SW_Push, SW49 SW_Push, SW5 SW_Push, SW50 SW_Push, SW51 SW_Push, SW52 SW_Push, SW53 SW_Push, SW54 SW_Push, SW55 SW_Push, SW56 SW_Push, SW57 SW_Push, SW58 SW_Push, SW59 SW_Push, SW6 SW_Push, SW60 SW_Push, SW61 SW_Push, SW62 SW_Push, SW63 SW_Push, SW64 SW_Push, SW65 SW_Push, SW66 SW_Push, SW67 SW_Push, SW7 SW_Push, SW8 SW_Push, SW9 SW_Push, U1 ATmega32U4-A, Y1 16MHz

Commit message: Update to new placement of Microcontroller
Parts:
- U1: moved to B.Cu
- moved C1 27.8 mm to (93.6, 119.5)
- moved SW1 25.3 mm to (92.0, 111.6)
- moved R1 20.6 mm to (116.2, 116.0)
- moved C3 17.7 mm to (94.6, 123.0), turned to 90 degrees
- moved C2 14.0 mm to (109.7, 107.8)
- moved R4 12.9 mm to (97.9, 109.5)
- moved C5 6.76 mm to (97.5, 123.7)
- moved C2 5.06 mm to (118.6, 117.2)
- moved U1 1.04 mm to (103.6, 116.8), turned to 45 degrees
Connections:
- D22 pad 1: COL1 -> ROW2
- D24 pad 2: COL1 -> ROW2
- D26 pad 1: COL1 -> ROW2
- D28 pad 2: COL1 -> ROW2
- D29 pad 1: COL1 -> ROW2
- D30 pad 2: COL1 -> ROW2
- D31 pad 1: COL1 -> ROW2
- D32 pad 2: COL1 -> ROW2
- D33 pad 1: COL1 -> ROW2
- D34 pad 2: COL1 -> ROW2
- D35 pad 1: COL1 -> ROW2
- D36 pad 2: COL1 -> ROW2
- D37 pad 1: COL1 -> ROW2
- D38 pad 2: COL1 -> ROW2
- U1 pad 30: COL1 -> ROW2
Routing:
- net COL1: track 695.9 -> 288.9 mm, vias 7 -> 4
- net ROW2: track 0.00 -> 338.8 mm, vias 0 -> 8
- net COL2: track 456.2 -> 403.6 mm, vias 5 -> 3
- net COL3: track 618.3 -> 582.0 mm, vias 5 -> 4
- net GND: track 466.5 -> 431.3 mm, vias 18 -> 16
- net COL5: track 341.5 -> 310.2 mm, vias 4 -> 3
- net COL4: track 585.9 -> 561.4 mm, vias 7 -> 8
- net COL6: track 354.0 -> 331.4 mm, vias 3 -> 4
- net COL0: track 336.1 -> 317.5 mm, vias 3 -> 2
- net Net-(U1-D+): track 231.3 -> 248.2 mm, vias 1 -> 0
- net ROW0: track 326.0 -> 310.9 mm, vias 12 -> 11
- net +5V: track 378.6 -> 366.6 mm
- net Net-(U1-D-): track 231.7 -> 243.3 mm, vias 1 -> 0
- net ROW4: track 376.7 -> 386.4 mm, vias 5 -> 6
- net Net-(U1-XTAL1): track 25.5 -> 19.9 mm, vias 1 -> 2
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