File: projects/Circuit Sax/src/MIDI Sax.kicad_pcb (KiCad board)
At the start: 2 copper layers, 105.4 x 215.6 mm, 75 parts, among them J1 Conn_01x17_Socket, J2 Conn_01x17_Socket, K1 SW_Push, K2 SW_Push, K3 SW_Push, K4 SW_Push, K5 SW_Push, K6 SW_Push, U1 MPXV5010GP

Commit message: Remove notes from PCB file
Other:
- board text removed: "I need to make sure the pins line up with the correct sockets also that the footprints for the through hole headers are correct also that the sensor footprint is correct, but seems like it is since its on the other side"
Changed lines of the file:
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@@
   (gr_line (start 151.884 166.74) (end 151.024 165.88)
     (stroke (width 0.25) (type solid)) (layer "F.SilkS"))
-  (gr_line (start 163.73 162.66) (end 163.73 162.16)
-    (stroke (width 0.15) (type default)) (layer "F.SilkS"))
-  (gr_line (start 167.73 166.66) (end 189.03 166.66)
-    (stroke (width 0.15) (type default)) (layer "F.SilkS"))
-  (gr_arc (start 167.73 166.66) (mid 164.901573 165.488427) (end 163.73 162.66)
-    (stroke (width 0.15) (type default)) (layer "F.SilkS"))
   (gr_line (start 85 200.001) (end 113.572 200.001)
     (stroke (width 0.1) (type default)) (layer "Edge.Cuts"))
@@
   (gr_line (start 124.672988 133.746334) (end 124.672988 140.459667)
     (stroke (width 0.1) (type default)) (layer "Edge.Cuts"))
-  (gr_text "I need to make sure the pins line up with the correct sockets\n\nalso that the footprints for the through hole headers are correct\n\nalso that the sensor footprint is correct, but seems like it is since its on the other side" (at -40 60) (layer "F.Cu")
-    (effects (font (size 1.5 1.5) (thickness 0.3) bold) (justify left bottom))
-  )
   (gr_text "Circuit Sax v1" (at 131.871 164.282) (layer "F.SilkS")
     (effects (font (size 1.5 1.5) (thickness 0.3) bold) (justify left top))
