File: projects/rgb_strip_controller/src/rgbcontroller.kicad_pcb (KiCad board)
At the start: 2 copper layers, 118.9 x 52.8 mm, 47 parts, among them J3 Barrel_Jack_Switch_Pin3Ring, J4 Conn_01x03_Pin, J5 Conn_01x03_Pin, J6 USB_B_Micro, Q1 BSS138, Q2 BSS138, Q3 BSS138, Q4 IRFZ44N, Q5 IRFZ44N, Q6 IRFZ44N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

Commit message: RGB_C
Parts:
- removed the G*** at (155.2, 105.4)
- removed the G*** at (155.0, 109.6)
- added G***: LOGO, kilibimg:instagramAcc-qr, F.Cu at (155.4, 108.8)
- added G***: LOGO, kilibimg:Telescope, B.Cu at (91.6, 109.6)
- added G***: LOGO, kilibimg:meth, B.Cu at (73.4, 119.2)
- added G***: LOGO, kilibimg:githubacc, B.Cu at (172.2, 115.6)
- C3, C4, C5: footprint Capacitor_SMD:C_0603_1608Metric -> Capacitor_SMD:C_0805_2012Metric_Pad1.18x1.45mm_HandSolder
- moved G*** 3.45 mm to (159.2, 89.2)
- moved G*** 3.17 mm to (98.9, 117.9), turned to 180 degrees
- moved C3 0.77 mm to (82.8, 116.4)
- moved G*** 0.72 mm to (156.0, 104.0)
- moved C4 0.60 mm to (82.8, 110.2)
Routing:
- net D5: track 57.9 -> 61.1 mm
- net 3.3V: track 278.3 -> 280.7 mm
- net RST: track 28.1 -> 29.9 mm
- net GND: track 302.9 -> 303.8 mm
- net DTR: track 107.7 -> 108.2 mm
Other:
- board text added: "Souptik"
- board text added: "heisenberg"
- board text added: "methamphetamine"
- board text removed: "@Souptik.me"
