File: projects/rgb_strip_controller/src/rgbcontroller.kicad_sch (KiCad schematic)
At the start: 42 parts, among them J3 Barrel_Jack_Switch_Pin3Ring, J4 Conn_01x03_Pin, J5 Conn_01x03_Pin, J6 USB_B_Micro, Q1 BSS138, Q2 BSS138, Q3 BSS138, Q4 IRFZ44N, Q5 IRFZ44N, Q6 IRFZ44N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

Commit message: RGB_C
Parts:
- C3, C4, C5: footprint Capacitor_SMD:C_0603_1608Metric -> Capacitor_SMD:C_0805_2012Metric_Pad1.18x1.45mm_HandSolder
Changed lines of the file:
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@@
 			)
 		)
-		(property "Footprint" "Capacitor_SMD:C_0603_1608Metric"
+		(property "Footprint" "Capacitor_SMD:C_0805_2012Metric_Pad1.18x1.45mm_HandSolder"
 			(at 73.3552 189.23 0)
 			(effects
@@
 			)
 		)
-		(property "Footprint" "Capacitor_SMD:C_0603_1608Metric"
+		(property "Footprint" "Capacitor_SMD:C_0805_2012Metric_Pad1.18x1.45mm_HandSolder"
 			(at 65.7352 189.23 0)
 			(effects
@@
 			)
 		)
-		(property "Footprint" "Capacitor_SMD:C_0603_1608Metric"
+		(property "Footprint" "Capacitor_SMD:C_0805_2012Metric_Pad1.18x1.45mm_HandSolder"
 			(at 78.74 108.9152 0)
 			(effects
