File: projects/Arduino_v1/arduino_v1/src/arduino_v1.kicad_pcb (KiCad board)
At the start: 2 copper layers, 55 x 70 mm, 36 parts, among them J1 Conn_01x06_Pin, J2 Conn_01x07_Pin, J3 Conn_01x08_Pin, J4 Conn_01x03_Pin, J5 USB_B, J6 Barrel_Jack_Switch, J7 Conn_01x08_Pin, U1 ATmega328-P, U2 LM7805_TO220, U3 CH340G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

Commit message: done
Parts:
- moved C10 44.5 mm to (40.8, 70.8)
- moved C7 44.5 mm to (60.6, 74.9)
- moved J5 44.5 mm to (60.9, 64.4)
- moved Y1 44.5 mm to (39.3, 93.2)
- moved C1 44.5 mm to (44.9, 97.7)
- moved C5 44.5 mm to (38.2, 116.0)
- moved D1 44.5 mm to (25.6, 66.7)
- moved D2 44.5 mm to (22.5, 97.7)
- moved G*** 44.5 mm to (43.2, 56.7)
- moved J4 44.5 mm to (51.0, 63.2)
- moved J7 44.5 mm to (17.9, 81.5)
- moved R1 44.5 mm to (22.5, 100.8)
- moved R2 44.5 mm to (39.3, 105.8)
- moved R4 44.5 mm to (47.9, 115.7)
- moved U1 44.5 mm to (33.7, 116.0)
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Routing:
- net VCC: track 121.9 -> 124.4 mm
- net D8: track 57.0 -> 56.0 mm, vias 3 -> 2
- net D5: vias 6 -> 3
- removed copper zone on B.Cu, net 5V
- removed copper zone on F.Cu, net GND
