File: projects/simonsaysskull/src/simon-says-skull.kicad_pcb (KiCad board)
At the start: 2 copper layers, 73 x 84 mm, 12 parts, among them SW1 SW_Push_LED, SW2 SW_Push_LED, SW3 SW_Push_LED, SW4 SW_Push_LED, SW5 SW_DPST_x2, U2 ATtiny85-20M

Commit message: Add files via upload
Routing:
- net GND: track 0.00 -> 189.8 mm
- net Net-(SW5A-B): track 0.00 -> 71.1 mm, vias 0 -> 1
- net Net-(BZ1-+): track 0.00 -> 66.0 mm
- net Net-(SW3-K): track 0.00 -> 48.8 mm, vias 0 -> 2
- net Net-(SW1-K): track 0.00 -> 45.8 mm
- net Net-(SW4-K): track 0.00 -> 26.9 mm
- net Net-(SW2-K): track 0.00 -> 22.9 mm
- net (no net): track 0.00 -> 8.20 mm
