File: projects/Koeg-Board/src/koeg-board-pcb.kicad_sch (KiCad schematic)
At the start: 0 parts

Commit message: Add files via upload
Parts:
- added BO1, BO2, BO3: break off, panelization:mouse-bite-2mm-slot, symbol Mechanical:MountingHole
- added FID1, FID2, FID3: Fiducial, Fiducial:Fiducial_1.5mm_Mask3mm, symbol Mechanical:Fiducial
Other:
- note added: "Fidutilas"
