File: projects/Koeg-Board/src/power.kicad_sch (KiCad schematic)
At the start: 9 parts, among them SW2 SW_On_Off, U11 BQ24075RGT

Commit message: Add files via upload
Parts:
- C87, C89, C91: LCSC (none) -> C307423
- R27: LCSC (none) -> C131467
- R29: LCSC (none) -> C25867
- R31: value 1.5k -> 4.7k; LCSC (none) -> C25940
- R33: value 1.5k -> 10k; LCSC (none) -> C25744
- U11: LCSC (none) -> C2865459
Changed lines of the file:
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@@
+			)
+		)
+		(property "LCSC" "C2865459"
+			(at 105.41 144.78 0)
+			(effects
+				(font
+					(size 1.27 1.27)
+				)
 			)
 		)
@@
 			)
 		)
+		(property "LCSC" "C307423"
+			(at 147.32 151.13 0)
+			(effects
+				(font
+					(size 1.27 1.27)
+				)
+				(hide yes)
+			)
+		)
 		(pin "1"
 		)
@@
 			)
 		)
+		(property "LCSC" "C25867"
+			(at 80.01 158.75 0)
+			(effects
+				(font
+					(size 1.27 1.27)
+				)
+				(hide yes)
+			)
+		)
 		(pin "2"
 		)
@@
 			)
 		)
-		(property "Value" "1.5k"
+		(property "Value" "4.7k"
 			(at 65.278 160.274 0)
 			(effects
@@
 		)
 		(property "Description" "Resistor"
+			(at 71.12 158.75 0)
+			(effects
+				(font
+					(size 1.27 1.27)
+				)
+				(hide yes)
+			)
+		)
+		(property "LCSC" "C25940"
 			(at 71.12 158.75 0)
 			(effects
@@
 			)
 		)
+		(property "LCSC" "C307423"
+			(at 132.08 151.13 0)
+			(effects
+				(font
+					(size 1.27 1.27)
+				)
+				(hide yes)
+			)
+		)
 		(pin "1"
 		)
@@
 		)
 		(property "Description" "Resistor"
+			(at 88.9 158.75 0)
+			(effects
+				(font
+					(size 1.27 1.27)
+				)
+				(hide yes)
+			)
+		)
+		(property "LCSC" "C131467"
 			(at 88.9 158.75 0)
 			(effects
@@
 			)
 		)
+		(property "LCSC" "C307423"
+			(at 59.69 149.86 0)
+			(effects
+				(font
+					(size 1.27 1.27)
+				)
+				(hide yes)
+			)
+		)
 		(pin "1"
 		)
@@
 			)
 		)
-		(property "Value" "1.5k"
+		(property "Value" "10k"
 			(at 127.762 152.146 0)
 			(effects
@@
 			(at 121.92 153.67 0)
 			(effects
+				(font
+					(size 1.27 1.27)
+				)
+				(hide yes)
+			)
+		)
+		(property "LCSC" "C25744"
+			(at 121.92 153.67 0)
+			(effects
