File: projects/Koeg-Board/src/side.kicad_sch (KiCad schematic)
At the start: 81 parts, among them J1 Conn_01x02, J2 SWD_Connector, J3 USB_C_Receptacle_USB2.0_16P, SW1 Reset Button, SW10 SW_Push, SW11 SW_Push, SW12 SW_Push, SW13 SW_Push, SW14 SW_Push, SW15 SW_Push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

Commit message: Add files via upload
Parts:
- added LOGO1: Logo_Open_Hardware_Small, koeg-logo:BM logo, symbol Graphic:Logo_Open_Hardware_Small
- added TP1: VSW, TestPoint:TestPoint_Pad_D2.0mm, symbol Connector:TestPoint
- added TP2: V_SYS, TestPoint:TestPoint_Pad_D2.0mm, symbol Connector:TestPoint
- added TP3: VBAT, TestPoint:TestPoint_Pad_D2.0mm, symbol Connector:TestPoint
- added TP4: GND, TestPoint:TestPoint_Pad_D2.0mm, symbol Connector:TestPoint
- C10, C19: LCSC (none) -> C1705
- C11, C12, C15, C31: LCSC (none) -> C106201
- C13: footprint Capacitor_SMD:C_0603_1608Metric -> Capacitor_SMD:C_0402_1005Metric; LCSC (none) -> C309455
- C14: footprint Capacitor_SMD:C_0603_1608Metric -> Capacitor_SMD:C_0402_1005Metric; LCSC (none) -> C327292
- C2: footprint Capacitor_SMD:C_0603_1608Metric -> Capacitor_SMD:C_0402_1005Metric; LCSC (none) -> C60474
- C39, C7: LCSC (none) -> C14445
- C4, C41, C43: LCSC (none) -> C60474
- C5: LCSC (none) -> C77177
- C6: LCSC (none) -> C107031
- C9: LCSC (none) -> C307423
- D10, D11, D12, D13, D14, D15, D16, D17, D18, D19, D2, D20, D21, D22, D3, D4, D5, D6, D7, D8, D9: LCSC (none) -> C963381
- J1, J2: now left out of the parts list
- L4: LCSC (none) -> C86065
- L5: LCSC (none) -> C86061
- R1: LCSC (none) -> C60491
- R2: LCSC (none) -> C3016043
- R3: LCSC (none) -> C11512
- R4, R5: LCSC (none) -> C25905
- SW1: LCSC (none) -> C2886897
- SW10, SW11, SW12, SW13, SW14, SW15, SW16, SW17, SW18, SW19, SW20, SW21, SW22, SW23, SW3, SW4, SW5, SW6, SW7, SW8, SW9: LCSC (none) -> C5333465
- U2: LCSC (none) -> C7519
- U7: LCSC C2895249 -> C2895249
- Y1: LCSC C2149238 -> C2149238
Connections:
- net GND: now also TP4.1
- net VBAT: now also TP3.1
- net VSW: now also TP1.1
- net V_SYS: now also TP2.1
Other:
- note added: "Test Points"
- moved on the sheet: AE65, C10, C11, C12, C13, C14, C19, C39, C4, C41, C43, C5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
