File: projects/esphome-han-reader/src/esphome-han-reader.kicad_sch (KiCad schematic)
At the start: 16 parts, among them J1 RJ12, J2 ProgammingPins, Q1 BC817W, SW1 ResetBtn, SW2 FlashBtn, U1 ESP-07, U2 LD1117S33CTR_SOT223

Commit message: feat: new src files
Connections:
- net +3V3: now also U2.2 (VO); no longer U2.3 (VI)
- net +5V: now also C1.2, U2.3 (VI); no longer C1.1, U2.2 (VO)
- net GND: now also C1.1; no longer C1.2
Other:
- moved on the sheet: C1, C2
