File: projects/Pico MMU Control Board/src/PicoMMUBoard.kicad_sch (KiCad schematic)
At the start: 29 parts, among them J1 USB_C, J2 PWR, J3 STLink, J4 TMC2209, J5 Servo Conn, J6 Conn_Stepper, SW1 RESET, SW2 BOOT, U1 USBLC6-2SC6, U2 AMS1117-3.3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

Commit message: Changes to layout
Parts:
- added C4, C5: 0.1uF, Capacitor_SMD:C_0603_1608Metric, symbol Device:C
- C13: footprint Capacitor_SMD:C_Elec_8x10.2 -> Capacitor_SMD:C_Elec_6.3x7.7
- SW1, SW2: footprint Button_Switch_SMD:SW_Push_TSB003A -> Button_Switch_SMD:SW4_KMS-P
Connections:
- net +3V3: now also C4.2
- net +5V: now also J5.2 (Pin_2), C5.1; no longer J5.1 (Pin_1)
- net GND: now also C4.1, C5.2
- net at U5.4 (B): now also J5.1 (Pin_1); no longer J5.2 (Pin_2)
