File: projects/Pico MMU Control Board/src/PicoMMUBoard.kicad_pcb (KiCad board)
At the start: 2 copper layers, 51.1 x 40.9 mm, 36 parts, among them J1 USB_C, J2 PWR, J3 STLink, J4 TMC2209, J5 Servo Conn, J6 Conn_Stepper, SW1 RESET, SW2 BOOT, U1 USBLC6-2SC6, U2 AMS1117-3.3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

Commit message: Changes to layout
Parts:
- added C4: 0.1uF, Capacitor_SMD:C_0603_1608Metric, F.Cu at (156.5, 74.2)
- added C5: 0.1uF, Capacitor_SMD:C_0603_1608Metric, F.Cu at (159.8, 74.2)
- SW1, SW2: footprint Button_Switch_SMD:SW_Push_TSB003A -> Button_Switch_SMD:SW4_KMS-P
- moved C9 6.15 mm to (143.0, 46.7), turned to -90 degrees
- moved R5 5.22 mm to (134.6, 46.7), turned to -90 degrees
- moved U5 3.05 mm to (158.0, 76.7)
- moved J2 2.79 mm to (130.8, 58.2)
- moved SW1 1.79 mm to (138.9, 45.8), turned to 180 degrees
- moved SW2 1.55 mm to (130.6, 45.9), turned to 180 degrees
- moved REF** 0.25 mm to (127.3, 84.1)
Connections:
- J5 pad 1: +5V -> Net-(J5-Pin_1)
- J5 pad 2: Net-(J5-Pin_2) -> +5V
- U5 pad 4: Net-(J5-Pin_2) -> Net-(J5-Pin_1)
Routing:
- net Net-(U4-NRST): track 38.8 -> 51.3 mm
- net Net-(U4-PB0): track 46.8 -> 56.4 mm
- net +3V3: track 138.3 -> 146.6 mm
- net Net-(J5-Pin_2): track 3.32 -> 0.00 mm
- net GND: track 20.0 -> 23.3 mm
- net Net-(J5-Pin_1): track 0.00 -> 3.11 mm
- net SERVO: track 12.3 -> 10.1 mm
- net VCC: track 41.3 -> 40.1 mm
- net STEP: track 27.6 -> 27.0 mm
- net DIR: track 28.6 -> 28.0 mm
Other:
- board text added: "BOOT"
- board text added: "GND"
- board text added: "PWM"
- board text added: "PWR"
- board text added: "RESET"

Commit message: Changes to layout
Parts:
- moved C9 0.14 mm to (143.0, 46.9)
- moved R5 0.14 mm to (134.6, 46.8)
- moved SW1 0.14 mm to (138.9, 46.0)
- moved SW2 0.14 mm to (130.6, 46.0)
Other:
- board text added: "3.3V"
- board text added: "5V"
- board text added: "CLK"
- board text added: "DIO"
- board text removed: "PWR"
