File: projects/HH-The-Nob/src/nob.kicad_pcb (KiCad board)
At the start: 2 copper layers, 70 x 70.6 mm, 49 parts, among them P0 Conn_01x01_Pin, P1 Conn_01x01_Pin, P1.5 Conn_01x01_Pin, P10 Conn_01x01_Pin, U1 XIAO-ESP32-C3-SMD, U2 AS5600

Commit message: update
Added holes to gerble
Routing:
- net BAT_P: vias 0 -> 3
Other:
- board text added: "JLCJLCJLCJLC"
Changed lines of the file:
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@@
+		)
+	)
+	(gr_text "JLCJLCJLCJLC"
+		(at 135.5 82.25 0)
+		(layer "B.SilkS")
+		(effects
+			(font
+				(size 1 1)
+				(thickness 0.1)
+			)
+			(justify left bottom mirror)
 		)
 	)
@@
 	)
 	(segment
-		(start 132.5 46.628)
-		(end 134.39 44.738)
-		(width 0.5)
-		(layer "B.Cu")
+		(start 133.413 44.738)
+		(end 133.4 44.725)
+		(width 0.5)
+		(layer "F.Cu")
 		(net 36)
 	)
-	(segment
-		(start 149.15 68.75)
+	(via
+		(at 135.425 44.725)
+		(size 0.6)
+		(drill 0.3)
+		(layers "F.Cu" "B.Cu")
+		(net 36)
+	)
+	(via
+		(at 134.39 44.738)
+		(size 0.6)
+		(drill 0.3)
+		(layers "F.Cu" "B.Cu")
+		(net 36)
+	)
+	(via
+		(at 133.4 44.725)
+		(size 0.6)
+		(drill 0.3)
+		(layers "F.Cu" "B.Cu")
+		(net 36)
+	)
+	(segment
+		(start 134.25 64.25)
 		(end 144.65 64.25)
 		(width 0.5)
@@
 	)
 	(segment
+		(start 134.387 44.738)
+		(end 132.5 46.625)
+		(width 0.5)
+		(layer "B.Cu")
+		(net 36)
+	)
+	(segment
+		(start 132.5 46.625)
+		(end 132.5 62.5)
+		(width 0.5)
+		(layer "B.Cu")
+		(net 36)
+	)
+	(segment
+		(start 134.39 44.738)
+		(end 134.387 44.738)
+		(width 0.5)
+		(layer "B.Cu")
+		(net 36)
+	)
+	(segment
 		(start 132.5 62.5)
-		(end 132.5 46.628)
+		(end 134.25 64.25)
 		(width 0.5)
 		(layer "B.Cu")
@@
 	(segment
 		(start 144.65 64.25)
-		(end 134.25 64.25)
-		(width 0.5)
-		(layer "B.Cu")
-		(net 36)
-	)
-	(segment
-		(start 134.25 64.25)
-		(end 132.5 62.5)
-		(width 0.5)
-		(layer "B.Cu")
+		(end 149.15 68.75)
+		(width 0.5)
+		(layer "B.Cu")

Commit message: Add files via upload
Parts:
- added G***: LOGO, MyLib:snowflake, B.Cu at (153.4, 56.5)
- added G***: LOGO, MyLib:snowflake, B.Cu at (103.0, 70.0)
- added G***: LOGO, MyLib:snowflake, B.Cu at (143.5, 93.4)
- added G***: LOGO, MyLib:snowflake, B.Cu at (106.6, 83.5)
- added G***: LOGO, MyLib:snowflake, B.Cu at (153.4, 83.5)
- added G***: LOGO, MyLib:snowflake, B.Cu at (106.6, 56.5)
- added G***: LOGO, MyLib:snowflake, B.Cu at (130.0, 97.0)
- added G***: LOGO, MyLib:snowflake, B.Cu at (116.5, 93.4)
- added G***: LOGO, MyLib:snowflake, B.Cu at (157.0, 70.0)
- moved BAT_N1 4.59 mm to (149.0, 71.0), turned to -90 degrees
- moved BAT_P1 1.61 mm to (149.0, 67.2), turned to -90 degrees
Routing:
- net BAT_P: track 37.8 -> 37.0 mm, vias 3 -> 0
