File: projects/souptik-hackyholiday/src/Hackholidays.kicad_pcb (KiCad board)
At the start: 2 copper layers, 50 x 90 mm, 71 parts, among them J1 DHT11, M1 MOUDLE-SEEEDUINO-XIAO

Commit message: Add files via upload
Parts:
- added J3: USB_C_Receptacle_USB2.0_16P, Connector_USB:USB_C_Receptacle_GCT_USB4105-xx-A_16P_TopMnt_Horizontal, F.Cu at (223.7, 34.5)
- moved G***17 17.5 mm to (210.3, 25.7)
- moved G***18 17.5 mm to (210.3, 25.7)
- moved G***15 6.75 mm to (220.7, 25.9)
- moved G***16 6.75 mm to (220.7, 25.9)
- moved G***1 0.76 mm to (214.1, 36.3)
- moved G***2 0.76 mm to (214.1, 36.3)
Routing:
- net GND: track 260.9 -> 323.5 mm
- net +5V: track 0.00 -> 24.4 mm, vias 0 -> 3
