File: projects/souptik-hackyholiday/src/Hackholidays.kicad_sch (KiCad schematic)
At the start: 33 parts, among them J1 DHT11, M1 MOUDLE-SEEEDUINO-XIAO

Commit message: Add files via upload
Parts:
- added J3: USB_C_Receptacle_USB2.0_16P, Connector_USB:USB_C_Receptacle_GCT_USB4105-xx-A_16P_TopMnt_Horizontal, symbol Connector:USB_C_Receptacle_USB2.0_16P
Connections:
- net +5V: now also J3.A4 (VBUS), J3.A9 (VBUS), J3.B4 (VBUS), J3.B9 (VBUS)
- net GND: now also J3.A1 (GND), J3.A12 (GND), J3.B1 (GND), J3.B12 (GND), J3.S1 (SHIELD)
- no-connect marks 0 -> 8
