File: projects/snowflake/src/snowflake.kicad_sch (KiCad schematic)
At the start: 50 parts, among them SW1 SW_Push, U1 XIAO-ESP32-C3-SMD

Commit message: update footprint + dad pcba
Parts:
- SW1: footprint Button_Switch_THT:SW_PUSH_6mm -> LCSC:SW-SMD_4P-L5.1-W5.1-P3.70-LS6.5-TL_H1.5
Changed lines of the file:
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@@
 			)
 		)
-		(property "Footprint" "Button_Switch_THT:SW_PUSH_6mm"
+		(property "Footprint" "LCSC:SW-SMD_4P-L5.1-W5.1-P3.70-LS6.5-TL_H1.5"
 			(at 195.58 127 0)
 			(effects
