File: projects/PCBProController/src/pcb_pro_controller.kicad_pcb (KiCad board)
At the start: 2 copper layers, 126.5 x 83 mm, 66 parts, among them J1 USB_C_Receptacle_USB2.0_16P, SW1 SW_PushHome, SW10 SW_PushScreenshot, SW11 SW_Push-, SW12 SW_PushLeft, SW13 SW_PushUp, SW14 SW_PushDown, SW15 SW_PushRight, SW16 SW_PushZL, SW2 SW_Push+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

Commit message: re updated
Parts:
- J1: footprint Connector_USB:USB_C_Receptacle_GCT_USB4085 -> Connector_USB:USB_C_Receptacle_G-Switch_GT-USB-7010ASV
- U1: value FT231XS-U -> FT231XS-R
- moved J1 5.46 mm to (203.5, 29.8)
Routing:
- net GND: track 147.2 -> 146.0 mm
- net D-: track 42.5 -> 43.8 mm
- net Net-(R22-Pad2): track 59.3 -> 60.3 mm
- net D+: track 37.2 -> 38.2 mm
- net +5V: track 11.1 -> 10.2 mm
