File: projects/PCBProController/src/pcb_pro_controller.kicad_sch (KiCad schematic)
At the start: 61 parts, among them J1 USB_C_Receptacle_USB2.0_16P, SW1 SW_PushHome, SW10 SW_PushScreenshot, SW11 SW_Push-, SW12 SW_PushLeft, SW13 SW_PushUp, SW14 SW_PushDown, SW15 SW_PushRight, SW16 SW_PushZL, SW2 SW_Push+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

Commit message: re updated
Parts:
- J1: footprint Connector_USB:USB_C_Receptacle_GCT_USB4085 -> Connector_USB:USB_C_Receptacle_G-Switch_GT-USB-7010ASV
- U1: value FT231XS-U -> FT231XS-R
Other:
- moved on the sheet: D1, D2, D3, D4, R1, R10, R12, R15, R16, R17, R18, R19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
