File: projects/tobydio/src/tobydio-pub.kicad_pcb (KiCad board)
At the start: 2 copper layers, 42.3 x 61.5 mm, 41 parts, among them J1 Conn_01x02_Pin, J10 Conn_01x03_Pin, J2 PJ-320D-A, J3 Conn_01x04_Pin, J5 Conn_01x01_Pin, J6 Conn_01x03_Pin, J7 Conn_01x04_Pin, J8 PJ-320D-A, J9 Conn_01x03_Pin, U1 PCM5100APWR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

Commit message: update source files for tobydio
Other:
- board text added: "there was some very emotional text here but i took it out heheheha"
- board text removed: "dear scarlett, you are over the best of what i could have wish for thank you so much for being a part of my life - toby"
