File: projects/tobydio/src/tobydio-pub-2.kicad_sch (KiCad schematic)
At the start: 41 parts, among them J1 Conn_01x02_Pin, J10 Conn_01x03_Pin, J2 PJ-320D-A, J3 Conn_01x04_Pin, J5 Conn_01x01_Pin, J6 Conn_01x03_Pin, J7 Conn_01x04_Pin, J8 PJ-320D-A, J9 Conn_01x03_Pin, U1 PCM5100APWR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

Commit message: newer board, using more basic parts to save money
Parts:
- removed C10, C16, C18, C8, C9: 10uF, Capacitor_SMD:CP_Elec_6.3x7.7, symbol Device:C_Polarized_US
- removed C22: 1uF, Capacitor_SMD:CP_Elec_4x5.4, symbol Device:C_Polarized_US
- added C10, C16, C8, C9: 10uF, Capacitor_SMD:C_0402_1005Metric_Pad0.74x0.62mm_HandSolder, symbol Device:C
- added C18: 10uF, Capacitor_SMD:C_0603_1608Metric_Pad1.08x0.95mm_HandSolder, symbol Device:C
- added C22: 2.2nF, Capacitor_SMD:C_0805_2012Metric_Pad1.18x1.45mm_HandSolder, symbol Device:C
- C1, C13, C15, C17, C2, C3, C4: LCSC Part # (none) -> C1525
- C11, C12, C21: footprint Capacitor_SMD:C_0402_1005Metric_Pad0.74x0.62mm_HandSolder -> Capacitor_SMD:C_0805_2012Metric_Pad1.18x1.45mm_HandSolder; LCSC Part # (none) -> C28260
- C14: footprint Capacitor_SMD:CP_Elec_6.3x7.7 -> Capacitor_SMD:C_0603_1608Metric_Pad1.08x0.95mm_HandSolder; symbol Device:C_Polarized_US -> Device:C; LCSC Part # (none) -> C19702
- C19: footprint Capacitor_SMD:CP_Elec_4x5.4 -> Capacitor_SMD:C_0805_2012Metric_Pad1.18x1.45mm_HandSolder; symbol Device:C_Polarized_US -> Device:C; LCSC Part # (none) -> C28323
- C20: value 2.2nF -> 1uF; footprint Capacitor_SMD:C_0402_1005Metric_Pad0.74x0.62mm_HandSolder -> Capacitor_SMD:C_0805_2012Metric_Pad1.18x1.45mm_HandSolder; LCSC Part # (none) -> C28323
- C5, C6: footprint Capacitor_SMD:C_0402_1005Metric_Pad0.74x0.62mm_HandSolder -> Capacitor_SMD:C_0603_1608Metric_Pad1.08x0.95mm_HandSolder; LCSC Part # (none) -> C23630
- C7: footprint Capacitor_SMD:CP_Elec_6.3x7.7 -> Capacitor_SMD:C_0402_1005Metric_Pad0.74x0.62mm_HandSolder; symbol Device:C_Polarized_US -> Device:C; LCSC Part # (none) -> C15525
- D1: LCSC Part # (none) -> C2297
- J1: footprint Connector_PinSocket_2.54mm:PinSocket_1x02_P2.54mm_Vertical -> Connector_PinHeader_2.54mm:PinHeader_1x02_P2.54mm_Vertical
- J10: footprint Connector_PinSocket_2.54mm:PinSocket_1x03_P2.54mm_Vertical -> Connector_PinHeader_2.54mm:PinHeader_1x03_P2.54mm_Vertical
- R1, R2, R3, R4: LCSC Part # (none) -> C25117
- R5: value 200 -> 220; footprint Resistor_SMD:R_0603_1608Metric_Pad0.98x0.95mm_HandSolder -> Resistor_SMD:R_0402_1005Metric_Pad0.72x0.64mm_HandSolder; LCSC Part # (none) -> C25091
Connections:
- net +3.3V: now also C16.1, C8.1, C9.1
- net GND: now also C10.2, C16.2, C18.2, C22.2, C8.2, C9.2; no longer C20.2
- net at C17.1, U2.1 (VREF): now also C18.1
- net at J7.3 (Pin_3), J8.3: now also C20.2
- net at R4.2: now also C20.1, C22.1; no longer C21.1
- net at C4.1, U1.18 (LDOO): now also C10.1
- net at C19.1, R3.2: now also C21.1; no longer C20.1
