File: projects/tobydio/src/tobydio.kicad_sch (KiCad schematic)
At the start: 41 parts, among them J1 Conn_01x02_Pin, J10 Conn_01x03_Pin, J2 PJ-320D-A, J3 Conn_01x04_Pin, J5 Conn_01x01_Pin, J6 Conn_01x03_Pin, J7 Conn_01x04_Pin, J8 PJ-320D-A, J9 Conn_01x03_Pin, U1 PCM5100APWR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

Commit message: update tobydio board
Other:
- company: (none) -> DaCloud
- title: (none) -> tobydio - pcm5100a and pcm1808 breakout board
- moved on the sheet: C11, C12, C21, C22
