File: projects/3DPrinterHeatBed/src/PCB.kicad_pcb (KiCad board)
At the start: 2 copper layers, 256 x 256 mm, 4 parts

Commit message: Add files via upload
Routing:
- net (no net): track 13725.4 -> 13215.2 mm
