File: projects/Wolf's megapad/src/megapad.kicad_sch (KiCad schematic)
At the start: 75 parts, among them SW1 MX1A-11NW, SW2 MX1A-11NW, SW3 MX1A-11NW, SW4 MX1A-11NW, SW5 MX1A-11NW, SW6 MX1A-11NW, U1 SL2.1A_C6798314, U2 TS3USB221RSER, U3 W25Q80DVSNIG, U4 ABM8-272-T3_C20625731, U5 RP2040, U6 NCP1117ST33T3G

Commit message: feat: cut down costs and update design files
Parts:
- removed C2, C3: 100uF, PCM_JLCPCB:C_1206, symbol PCM_JLCPCB-Capacitors:1206,100uF
- removed D1, D2, D3, D4, D5: DS34W-MS, easyeda2kicad:SOD-123FL_L2.8-W1.8-LS3.7-RD, symbol easyeda2kicad:DS34W-MS
- added Q1, Q2, Q3, Q4, Q5: AO3415AL, easyeda2kicad:SOT-23-3_L2.9-W1.6-P1.90-LS2.9-BL, symbol easyeda2kicad:AO3415AL
- added R21, R22, R23, R24, R25: 100kΩ, PCM_JLCPCB:R_0402, symbol PCM_JLCPCB-Resistors:0402,100kΩ
- DirectPWR1: value FC-F1005BK-470G5 -> FC-F1005WD-455K5; symbol easyeda2kicad:FC-F1005BK-470G5 -> easyeda2kicad:FC-F1005WD-455K5; LCSC Part C130724 -> C130725
- HubPWR1: value FC-F1005UGK-520M5 -> FC-F1005WD-455K5; footprint easyeda2kicad:LED0402-RD -> easyeda2kicad:LED0402-R-RD; symbol easyeda2kicad:FC-F1005UGK-520M5 -> easyeda2kicad:FC-F1005WD-455K5; LCSC Part C130723 -> C130725
- HubUSBA1: footprint easyeda2kicad:USB-A-TH_AF-10.0-HC6.3 -> easyeda2kicad:USB-A-SMD_C39429; symbol easyeda2kicad:AF10.0HC6.3 -> easyeda2kicad:USB-AF-90-10X14.4-H6.57; LCSC Part C456017 -> C39429
- R2, R3, R4, R5: footprint PCM_JLCPCB:R_0402 -> PCM_JLCPCB:R_0603; symbol PCM_JLCPCB-Resistors:0402,56kΩ -> PCM_JLCPCB-Resistors:0603,56kΩ; Class Preferred Component -> Basic Component; LCSC C25796 -> C23206; Overload Voltage (Max) 50V -> 75V; Part 0402WGF5602TCE -> 0603WAF5602T5E; Power(Watts) 62.5mW -> 100mW; Stock 318475 -> 232123
- U4: value ABM8-272-T3_C20625731 -> X322512MSB4SI; footprint easyeda2kicad:CRYSTAL-SMD_4P-L3.2-W2.5-BL -> PCM_JLCPCB:CRYSTAL-SMD_4P-L3.2-W2.5-BL; symbol easyeda2kicad:ABM8-272-T3_C20625731 -> PCM_JLCPCB-Crystals:Crystal, 12MHz, 20pF; Attrition Qty (none) -> 4; Category (none) -> Crystals/Oscillators/Resonators,Crystals; Class (none) -> Basic Component; Crystal Type (none) -> SMD Crystal Resonator; Frequency (none) -> 12MHz; Frequency Stability (none) -> ±20ppm; Frequency Tolerance (none) -> ±10ppm; LCSC (none) -> C9002; Load Capacitance (none) -> 20pF; Manufacturer (none) -> Yangxing Tech; Minimum Qty (none) -> 5; Normal Temperature Frequency Tolerance (none) -> ±10ppm; Operating Temperature (none) -> -40°C~+85°C; Part (none) -> X322512MSB4SI; Price (none) -> 0.069USD; Process (none) -> SMT; Stock (none) -> 98766; Type (none) -> Surface Mount Crystal
Connections:
- net +5V: now also C1.2, C4.2, C5.2, Q1.3 (D), Q2.3 (D), Q3.2 (S), Q4.2 (S), Q5.2 (S)
- net 5VDET: now also Q1.2 (S)
- net GND: now also HubPWR1.2 (K), HubUSBA1.0 (SHELD), R21.1, R22.1, R23.1, R24.1, R25.1; no longer HubPWR1.1 (K), HubUSBA1.5 (SHELL), HubUSBA1.6 (SHELL)
- net at HubUSBA1.1 (VCC): now also Q3.3 (D); no longer C1.2
- net at HubUSBC1.A4 (VBUS), HubUSBC1.A9 (VBUS): now also Q4.3 (D); no longer C4.2
- net at HubUSBC2.A4 (VBUS), HubUSBC2.A9 (VBUS): now also Q5.3 (D); no longer C5.2
- net at F2.2, R13.1: now also Q2.2 (S)
- net at R7.2: now also HubPWR1.1 (A); no longer HubPWR1.2 (A)
- new net: Q4.1 (G), R24.2
- new net: Q5.1 (G), R25.2
- new net: Q3.1 (G), R23.2
- new net: Q1.1 (G), R21.2
- new net: Q2.1 (G), R22.2
Other:
- moved on the sheet: C1, C11, C4, C5, C8, HubUSBC1, HubUSBC2, R2, R3, R4, R5

Commit message: feat: update megapad design and schematic
Parts:
- removed C11: 100nF, PCM_JLCPCB:C_0402, symbol PCM_JLCPCB-Capacitors:0402,100nF
- removed DirectPWR1: FC-F1005WD-455K5, easyeda2kicad:LED0402-R-RD, symbol easyeda2kicad:FC-F1005WD-455K5
- removed F2: SMD1206P150TF, easyeda2kicad:F1206, symbol easyeda2kicad:SMD1206P150TF
- removed Q1, Q2, Q3, Q4, Q5: AO3415AL, easyeda2kicad:SOT-23-3_L2.9-W1.6-P1.90-LS2.9-BL, symbol easyeda2kicad:AO3415AL
- removed R11, R8: 5.1kΩ, PCM_JLCPCB:R_0402, symbol PCM_JLCPCB-Resistors:0402,5.1kΩ
- removed R12, R14: 10kΩ, PCM_JLCPCB:R_0402, symbol PCM_JLCPCB-Resistors:0402,10kΩ
- removed R13: 200Ω, PCM_JLCPCB:R_0402, symbol PCM_JLCPCB-Resistors:0402,200Ω
- removed R21, R22, R23, R24, R25: 100kΩ, PCM_JLCPCB:R_0402, symbol PCM_JLCPCB-Resistors:0402,100kΩ
- removed RP2040Upstream1: USB3.1C16PFSMT, easyeda2kicad:USB-C-SMD_TYPE-C-USB-17, symbol easyeda2kicad:USB3.1C16PFSMT
- removed U2: TS3USB221RSER, easyeda2kicad:UQFN-10_L2.0-W1.5-P0.50-BL, symbol easyeda2kicad:TS3USB221RSER
- added D1, D2, D3, D4: TPD2E2U06DCKR, easyeda2kicad:SC-70-3_L2.0-W1.3-P0.65-LS2.1-BL, symbol easyeda2kicad:TPD2E2U06DCKR
- HubUSBA1: value AF 10.0 HC6.3 -> USB-AF-90-10X14.4-H6.57
- HubUSBC1, HubUSBC2, HubUpstream1: value USB3.1C16PFSMT -> MC-311D; footprint easyeda2kicad:USB-C-SMD_TYPE-C-USB-17 -> easyeda2kicad:USB-C-SMD_MC-311D; symbol easyeda2kicad:USB3.1C16PFSMT -> easyeda2kicad:MC-311D; LCSC Part C167321 -> C136423
- R14: renamed from R19; value 200Ω -> 47Ω; footprint PCM_JLCPCB:R_0402 -> PCM_JLCPCB:R_0603; symbol PCM_JLCPCB-Resistors:0402,200Ω -> PCM_JLCPCB-Resistors:0603,47Ω; LCSC C25087 -> C23182; Overload Voltage (Max) 50V -> 75V; Part 0402WGF2000TCE -> 0603WAF470JT5E; Power(Watts) 62.5mW -> 100mW; Resistance 200Ω -> 47Ω; Stock 512249 -> 1226635
- R15: renamed from R20; value 200Ω -> 47Ω; footprint PCM_JLCPCB:R_0402 -> PCM_JLCPCB:R_0603; symbol PCM_JLCPCB-Resistors:0402,200Ω -> PCM_JLCPCB-Resistors:0603,47Ω; LCSC C25087 -> C23182; Overload Voltage (Max) 50V -> 75V; Part 0402WGF2000TCE -> 0603WAF470JT5E; Power(Watts) 62.5mW -> 100mW; Resistance 200Ω -> 47Ω; Stock 512249 -> 1226635
- R7: value 200Ω -> 150Ω; footprint PCM_JLCPCB:R_0402 -> PCM_JLCPCB:R_0805; symbol PCM_JLCPCB-Resistors:0402,200Ω -> PCM_JLCPCB-Resistors:0805,150Ω; LCSC C25087 -> C17471; Overload Voltage (Max) 50V -> 150V; Part 0402WGF2000TCE -> 0805W8F1500T5E; Power(Watts) 62.5mW -> 125mW; Price 0.004USD -> 0.005USD; Resistance 200Ω -> 150Ω; Stock 512249 -> 430960
- U3: renamed from U4; value X322512MSB4SI -> ABM8-272-T3_C20625731; footprint PCM_JLCPCB:CRYSTAL-SMD_4P-L3.2-W2.5-BL -> easyeda2kicad:CRYSTAL-SMD_4P-L3.2-W2.5-BL; symbol PCM_JLCPCB-Crystals:Crystal, 12MHz, 20pF -> easyeda2kicad:ABM8-272-T3_C20625731
- renumbered C14 to C11, C15 to C12, C16 to C13, C17 to C14, C18 to C15, C19 to C16, C20 to C17, C21 to C18, C22 to C19, C6 to C2, C23 to C20, C24 to C21, C25 to C22, C7 to C3, C8 to C6, C12 to C7, C9 to C8, C13 to C9, R15 to R10, R16 to R11, R17 to R12, R18 to R13, R6 to R4, R4 to R5, R5 to R6, R9 to R8, R10 to R9, U6 to U2, U3 to U4
Connections:
- net 5VDET is gone; now on net +5V: F1.2, R7.1
- net +5V: now also HubUSBA1.1 (VCC), HubUSBC1.A4-B9 (VBUS), HubUSBC1.B4-A9 (VBUS), HubUSBC2.A4-B9 (VBUS), HubUSBC2.B4-A9 (VBUS)
- net D+: now also D1.1 (IO1)
- net D-: now also D1.2 (IO2)
- net GND: now also HubUSBA1.5 (SHELD), HubUSBA1.6 (SHELD), HubUSBC1.1 (SHIELD), HubUSBC1.2 (SHIELD), HubUSBC1.3 (SHIELD), HubUSBC1.4 (SHIELD), HubUSBC1.A1-B12 (GND), HubUSBC1.B1-A12 (GND), HubUSBC2.1 (SHIELD), HubUSBC2.2 (SHIELD), HubUSBC2.3 (SHIELD), HubUSBC2.4 (SHIELD), HubUSBC2.A1-B12 (GND), HubUSBC2.B1-A12 (GND), HubUpstream1.1 (SHIELD), HubUpstream1.2 (SHIELD), HubUpstream1.3 (SHIELD), HubUpstream1.4 (SHIELD), HubUpstream1.A1-B12 (GND), HubUpstream1.B1-A12 (GND), D1.3 (GND), D2.3 (GND), D3.3 (GND), D4.3 (GND); no longer HubUSBA1.0 (SHELD), HubUSBC1.0, HubUSBC1.A1 (GND), HubUSBC1.A12 (GND), HubUSBC2.0, HubUSBC2.A1 (GND), HubUSBC2.A12 (GND), HubUpstream1.0, HubUpstream1.A1 (GND), HubUpstream1.A12 (GND)
- net HubRP2040+: now also R11.1
- net HubRP2040-: now also R12.1
- net HubUSBA1+: now also D2.2 (IO2)
- net HubUSBA1-: now also D2.1 (IO1)
- net HubUSBC1+: now also D4.2 (IO2)
- net HubUSBC1-: now also D4.1 (IO1)
- net HubUSBC2+: now also D3.2 (IO2)
- net HubUSBC2-: now also D3.1 (IO1)
- net VBUS: now also HubUpstream1.A4-B9 (VBUS), HubUpstream1.B4-A9 (VBUS); no longer HubUpstream1.A4 (VBUS), HubUpstream1.A9 (VBUS)
- net at R4.2: now also HubUpstream1.B5 (CC2); no longer HubUpstream1.A5 (CC1)
- net at R3.2: now also HubUSBC2.A5 (CC1); no longer HubUSBC2.B5 (CC2)
- net at R1.2: now also HubUpstream1.A5 (CC1); no longer HubUpstream1.B5 (CC2)
- net at R6.2: now also HubUSBC2.B5 (CC2); no longer HubUSBC2.A5 (CC1)
- net at R2.2: now also HubUSBC1.A5 (CC1); no longer HubUSBC1.B5 (CC2)
- net at R5.2: now also HubUSBC1.B5 (CC2); no longer HubUSBC1.A5 (CC1)
- no-connect marks 28 -> 26
Other:
- note added: "ESD protection"
- note removed: "RP2040 direct connection port"
- note removed: "These two port is not intended to conenct simultaneously USB Hub one will power RP2040 as well downstream ports Where RP2040 direct one will power RP2040 only"
- moved on the sheet: BOOT1, C11, C12, C13, C14, C15, C16, C17, C18, C19, C20, C21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
